Commit message: added sensors to the robot: camera and laser all working

File: src/mybot_description/urdf/mybot.xacro (robot description, xacro)
@@ -1,4 +1,7 @@
 <?xml version='1.0'?>
 <robot name="myrobot" xmlns:xacro="http://www.ros.org/wiki/xacro">
+<!--adding a camera basic properties-->
+  <xacro:property name="cameraSize" value="0.05"/>
+  <xacro:property name="cameraMass" value="0.1"/>
   <xacro:include filename="$(find mybot_description)/urdf/mybot.gazebo" />
   <xacro:include filename="$(find mybot_description)/urdf/materials.xacro" />
@@ -25,4 +28,5 @@
         <box size=".4 .2 .1"/>
       </geometry>
+      <material name="orange"/>
     </visual>
     <collision name='caster_collision'>
@@ -62,4 +66,5 @@
         <cylinder radius="0.1" length="0.05"/>
       </geometry>
+      <material name="black"/>
     </visual>
     <inertial>
@@ -86,4 +91,5 @@
         <cylinder radius="0.1" length="0.05"/>
       </geometry>
+      <material name="black"/>
     </visual>
     <inertial>
@@ -114,3 +120,58 @@
     <joint_properties damping="0.0" friction="0.0"/>
   </joint>
+<!-- adding camera link and joint-->
+  <link name="camera">
+    <collision><!--hitbox-->
+      <origin xyz="0 0 0" rpy="0 0 0"/> <!--cartesian and angular coord to place camera-->
+      <geometry>
+        <box size="${cameraSize} ${cameraSize} ${cameraSize}"/>
+      </geometry>
+    </collision>
+    <visual><!--how is it gonna look (smaller than hitbox-->
+      <origin xyz="0 0 0" rpy="0 0 0"/>
+      <geometry>
+        <box size="${cameraSize} ${cameraSize} ${cameraSize}"/>
+      </geometry>
+      <material name="green"/><!--what color is gonna be-->
+    </visual>
+    <inertial><!--physics!!!!-->
+      <mass value="${cameraMass}"/>
+      <origin xyz="0 0 0" rpy="0 0 0"/>
+      <box_inertia m="${cameraMass}" x="${cameraSize}" y="${cameraSize}" z="${cameraSize}"/>
+      <inertia ixx="1e-6" ixy="0" ixz="0" iyy="1e-6" iyz="0" izz="1e-6"/>
+    </inertial>
+  </link>
+  <joint name="camera_joint" type="fixed">
+    <axis xyz="0 1 0"/>
+    <origin xyz=".2 0 0" rpy="0 0 0"/>
+    <parent link="chassis"/> <!--takes chasis as model-->
+    <child link="camera"/>
+  </joint>
+<!--adding laser and the joint-->
+  <joint name="hokuyo_joint" type="fixed">
+    <axis xyz="0 1 0" />
+    <origin xyz=".15 0 .1" rpy="0 0 0"/>
+    <parent link="chassis"/>
+    <child link="hokuyo"/>
+  </joint>
+  <!-- Hokuyo Laser -->
+  <link name="hokuyo">
+    <collision>
+      <origin xyz="0 0 0" rpy="0 0 0"/>
+      <geometry>
+    <box size="0.1 0.1 0.1"/>
+      </geometry>
+    </collision>
+    <visual>
+      <origin xyz="0 0 0" rpy="0 0 0"/>
+      <geometry><!--for more complex geometries dae files with autocad-->
+        <mesh filename="package://mybot_description/meshes/hokuyo.dae"/>
+      </geometry>
+    </visual>
+    <inertial>
+      <mass value="1e-5" />
+      <origin xyz="0 0 0" rpy="0 0 0"/>
+      <inertia ixx="1e-6" ixy="0" ixz="0" iyy="1e-6" iyz="0" izz="1e-6" />
+    </inertial>
+</link>
 </robot>
